File: pcb/_autosave-CoquiKeyboard.sch (KiCad schematic (older format))
At the start: 116 parts

Commit message: more reformatting
Connections:
- wire segments 166 -> 181
Other:
- moved on the sheet: MX?
Changed lines of the file:
@@
 L MX_Alps_Hybrids:MX-1U MX?
 U 1 1 5CE8B73F
-P 2775 5100
-F 0 "MX?" H 2861 5317 60  0000 C CNN
-F 1 "MX-1U" H 2861 5243 20  0000 C CNN
-F 2 "" H 2750 5075 60  0001 C CNN
-F 3 "" H 2750 5075 60  0001 C CNN
-	1    2775 5100
+P 2800 5100
+F 0 "MX?" H 2886 5317 60  0000 C CNN
+F 1 "MX-1U" H 2886 5243 20  0000 C CNN
+F 2 "" H 2775 5075 60  0001 C CNN
+F 3 "" H 2775 5075 60  0001 C CNN
+	1    2800 5100
 	1    0    0    -1
 $EndComp
@@
 L MX_Alps_Hybrids:MX-1U MX?
 U 1 1 5CE8BF31
-P 3075 5100
-F 0 "MX?" H 3161 5317 60  0000 C CNN
-F 1 "MX-1U" H 3161 5243 20  0000 C CNN
-F 2 "" H 3050 5075 60  0001 C CNN
-F 3 "" H 3050 5075 60  0001 C CNN
-	1    3075 5100
+P 3100 5100
+F 0 "MX?" H 3186 5317 60  0000 C CNN
+F 1 "MX-1U" H 3186 5243 20  0000 C CNN
+F 2 "" H 3075 5075 60  0001 C CNN
+F 3 "" H 3075 5075 60  0001 C CNN
+	1    3100 5100
 	1    0    0    -1
 $EndComp
@@
 L MX_Alps_Hybrids:MX-1U MX?
 U 1 1 5CE8CC1A
-P 3375 5100
-F 0 "MX?" H 3461 5317 60  0000 C CNN
-F 1 "MX-1U" H 3461 5243 20  0000 C CNN
-F 2 "" H 3350 5075 60  0001 C CNN
-F 3 "" H 3350 5075 60  0001 C CNN
-	1    3375 5100
+P 3400 5100
+F 0 "MX?" H 3486 5317 60  0000 C CNN
+F 1 "MX-1U" H 3486 5243 20  0000 C CNN
+F 2 "" H 3375 5075 60  0001 C CNN
+F 3 "" H 3375 5075 60  0001 C CNN
+	1    3400 5100
 	1    0    0    -1
 $EndComp
@@
 L MX_Alps_Hybrids:MX-1U MX?
 U 1 1 5CEB9A42
-P 3675 5100
-F 0 "MX?" H 3761 5317 60  0000 C CNN
-F 1 "MX-1U" H 3761 5243 20  0000 C CNN
-F 2 "" H 3650 5075 60  0001 C CNN
-F 3 "" H 3650 5075 60  0001 C CNN
-	1    3675 5100
+P 3700 5100
+F 0 "MX?" H 3786 5317 60  0000 C CNN
+F 1 "MX-1U" H 3786 5243 20  0000 C CNN
+F 2 "" H 3675 5075 60  0001 C CNN
+F 3 "" H 3675 5075 60  0001 C CNN
+	1    3700 5100
 	1    0    0    -1
 $EndComp
@@
 L MX_Alps_Hybrids:MX-1U MX?
 U 1 1 5CEB9FDA
-P 3975 5100
-F 0 "MX?" H 4061 5317 60  0000 C CNN
-F 1 "MX-1U" H 4061 5243 20  0000 C CNN
-F 2 "" H 3950 5075 60  0001 C CNN
-F 3 "" H 3950 5075 60  0001 C CNN
-	1    3975 5100
+P 4000 5100
+F 0 "MX?" H 4086 5317 60  0000 C CNN
+F 1 "MX-1U" H 4086 5243 20  0000 C CNN
+F 2 "" H 3975 5075 60  0001 C CNN
+F 3 "" H 3975 5075 60  0001 C CNN
+	1    4000 5100
 	1    0    0    -1
 $EndComp
@@
 L MX_Alps_Hybrids:MX-1U MX?
 U 1 1 5CEBA483
-P 4275 5100
-F 0 "MX?" H 4361 5317 60  0000 C CNN
-F 1 "MX-1U" H 4361 5243 20  0000 C CNN
-F 2 "" H 4250 5075 60  0001 C CNN
-F 3 "" H 4250 5075 60  0001 C CNN
-	1    4275 5100
+P 4300 5100
+F 0 "MX?" H 4386 5317 60  0000 C CNN
+F 1 "MX-1U" H 4386 5243 20  0000 C CNN
+F 2 "" H 4275 5075 60  0001 C CNN
+F 3 "" H 4275 5075 60  0001 C CNN
+	1    4300 5100
 	1    0    0    -1
 $EndComp
@@
 L MX_Alps_Hybrids:MX-1U MX?
 U 1 1 5CEFCBC8
-P 4575 5100
-F 0 "MX?" H 4661 5317 60  0000 C CNN
-F 1 "MX-1U" H 4661 5243 20  0000 C CNN
-F 2 "" H 4550 5075 60  0001 C CNN
-F 3 "" H 4550 5075 60  0001 C CNN
-	1    4575 5100
+P 4600 5100
+F 0 "MX?" H 4686 5317 60  0000 C CNN
+F 1 "MX-1U" H 4686 5243 20  0000 C CNN
+F 2 "" H 4575 5075 60  0001 C CNN
+F 3 "" H 4575 5075 60  0001 C CNN
+	1    4600 5100
 	1    0    0    -1
 $EndComp
@@
 L MX_Alps_Hybrids:MX-1U MX?
 U 1 1 5CEFDBC9
-P 5175 5100
-F 0 "MX?" H 5261 5317 60  0000 C CNN
-F 1 "MX-1U" H 5261 5243 20  0000 C CNN
-F 2 "" H 5150 5075 60  0001 C CNN
-F 3 "" H 5150 5075 60  0001 C CNN
-	1    5175 5100
+P 5200 5100
+F 0 "MX?" H 5286 5317 60  0000 C CNN
+F 1 "MX-1U" H 5286 5243 20  0000 C CNN
+F 2 "" H 5175 5075 60  0001 C CNN
+F 3 "" H 5175 5075 60  0001 C CNN
+	1    5200 5100
 	1    0    0    -1
 $EndComp
@@
 L MX_Alps_Hybrids:MX-1.75U MX?
 U 1 1 5CF7D59E
-P 4875 5100
-F 0 "MX?" H 4961 5317 60  0000 C CNN
-F 1 "MX-1.75U" H 4961 5243 20  0000 C CNN
-F 2 "" H 4850 5075 60  0001 C CNN
-F 3 "" H 4850 5075 60  0001 C CNN
-	1    4875 5100
+P 4900 5100
+F 0 "MX?" H 4986 5317 60  0000 C CNN
+F 1 "MX-1.75U" H 4986 5243 20  0000 C CNN
+F 2 "" H 4875 5075 60  0001 C CNN
+F 3 "" H 4875 5075 60  0001 C CNN
+	1    4900 5100
 	1    0    0    -1
 $EndComp
@@
 	2400 5275 2475 5275
 Wire Wire Line
-	2675 5300 2675 5275
-Wire Wire Line
 	2675 5275 2750 5275
 Wire Wire Line
-	2975 5300 2975 5275
-Wire Wire Line
 	2975 5275 3050 5275
 Wire Wire Line
@@
 	4475 5275 4550 5275
 Wire Wire Line
-	4475 5275 4475 5300
-Wire Wire Line
-	4250 5275 4175 5275
-Wire Wire Line
-	4175 5275 4175 5300
+	2075 4325 2075 5075
+Connection ~ 2075 5075
+Wire Wire Line
+	2075 5075 2075 5825
+Connection ~ 2075 5825
+Wire Wire Line
+	2075 5825 2075 6575
+Wire Wire Line
+	2375 4325 2375 5075
+Connection ~ 2375 5075
+Wire Wire Line
+	2375 5075 2375 5825
+Connection ~ 2375 5825
+Wire Wire Line
+	2375 5825 2375 6575
+Wire Wire Line
+	2675 4325 2675 5075
+Wire Wire Line
+	2675 5500 2675 5825
+Connection ~ 2675 5075
+Wire Wire Line
+	2675 5075 2675 5275
+Connection ~ 2675 5275
+Wire Wire Line
+	2675 5275 2675 5300
+Connection ~ 2675 5825
+Wire Wire Line
+	2675 5825 2675 6575
+Wire Wire Line
+	2975 4325 2975 5075
+Wire Wire Line
+	2975 5500 2975 5825
+Connection ~ 2975 5275
+Wire Wire Line
+	2975 5275 2975 5300
+Connection ~ 2975 5825
+Wire Wire Line
+	2975 5825 2975 6575
+Wire Wire Line
+	3275 4325 3275 5075
+Wire Wire Line
+	3275 5500 3275 5825
+Connection ~ 3275 5825
+Wire Wire Line
+	3275 5825 3275 6575
+Connection ~ 2975 5075
+Wire Wire Line
+	2975 5075 2975 5275
+Connection ~ 3275 5075
+Wire Wire Line
+	3275 5075 3275 5300
 $EndSCHEMATC
