File: pcb/CoquiKeyboard.kicad_pcb (KiCad board)
At the start: 2 copper layers, 116 parts, among them SW1 SW_Push, U1 ATmega32U4-MU, Y1 16MHz

Commit message: fix keysize error
Parts:
- moved C4 494.2 mm to (-251.0, -29.9), turned to 180 degrees
- moved D30 488.7 mm to (-248.6, -26.8), turned to 180 degrees
- moved D10 488.4 mm to (-245.0, -47.7), turned to 180 degrees
- moved D32 487.9 mm to (-248.6, -23.4), turned to 180 degrees
- moved C2 485.5 mm to (-246.6, -29.9), turned to 180 degrees
- moved U1 482.2 mm to (-243.6, -38.8), turned to 180 degrees
- moved D9 478.6 mm to (-239.3, -51.0), turned to 180 degrees
- moved USB1 478.1 mm to (-244.3, -16.6), turned to 180 degrees
- moved D31 477.3 mm to (-242.9, -26.8), turned to 180 degrees
- moved D13 477.2 mm to (-239.3, -47.7), turned to 180 degrees
- moved R2 476.8 mm to (-235.8, -60.9), turned to 180 degrees
- moved C1 476.8 mm to (-242.2, -29.9), turned to 180 degrees
- moved D33 476.5 mm to (-242.9, -23.4), turned to 180 degrees
- moved D22 476.4 mm to (-236.5, -57.7), turned to 180 degrees
- moved D23 474.8 mm to (-236.5, -54.4), turned to 180 degrees
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
Commit message: arrange switches to keyboard layout
Parts:
- removed D44: SOD-123, Diode_SMD:D_SOD-123
- removed MX44: MX-1U, MX_Alps_Hybrid:MX-1U
- added D51: SOD-123, Diode_SMD:D_SOD-123, F.Cu at (33.5, 5.11)
- added MX51: MX-1U, MX_Alps_Hybrid:MX-1U, F.Cu at (299.0, 41.9)
- MX14, MX38, MX49, MX6: value MX-1U -> MX-1.25U; footprint MX_Alps_Hybrid:MX-1U -> MX_Alps_Hybrid:MX-1.25U
- MX15, MX39, MX47, MX7: value MX-1.25U -> MX-1U; footprint MX_Alps_Hybrid:MX-1.25U -> MX_Alps_Hybrid:MX-1U
- MX19: value MX-2.25U -> MX-1U; footprint MX_Alps_Hybrid:MX-2.25U -> MX_Alps_Hybrid:MX-1U
- MX21: value MX-1U -> MX-2.25U; footprint MX_Alps_Hybrid:MX-1U -> MX_Alps_Hybrid:MX-2.25U
- MX29: value MX-2.75U -> MX-1U; footprint MX_Alps_Hybrid:MX-2.75U -> MX_Alps_Hybrid:MX-1U
- MX3: value MX-1.5U -> MX-1.75U; footprint MX_Alps_Hybrid:MX-1.5U -> MX_Alps_Hybrid:MX-1.75U
- MX31: value MX-1U -> MX-2.75U; footprint MX_Alps_Hybrid:MX-1U -> MX_Alps_Hybrid:MX-2.75U
- MX45: value MX-1.75U -> MX-1U; footprint MX_Alps_Hybrid:MX-1.75U -> MX_Alps_Hybrid:MX-1U
- MX48: value MX-1U -> MX-1.75U; footprint MX_Alps_Hybrid:MX-1U -> MX_Alps_Hybrid:MX-1.75U
- U1: footprint Package_QFP:LQFP-44_10x10mm_P0.8mm -> Package_QFP:TQFP-48-1EP_7x7mm_P0.5mm_EP3.5x3.5mm
- moved USB1 483.6 mm to (231.6, -102.4), turned to 0 degrees
- moved U1 482.4 mm to (233.0, -113.3), turned to 0 degrees
- moved R2 473.9 mm to (237.4, -85.8), turned to 0 degrees
- moved D30 463.6 mm to (212.3, -77.0), turned to 0 degrees
- moved R3 459.1 mm to (228.9, -79.4), turned to 0 degrees
- moved D27 458.7 mm to (226.6, -89.3), turned to 0 degrees
- moved D17 458.0 mm to (226.6, -82.6), turned to 0 degrees
- moved D18 458.0 mm to (232.3, -89.3), turned to 0 degrees
- moved D5 454.8 mm to (223.8, -77.0), turned to 0 degrees
- moved D20 452.6 mm to (232.3, -82.6), turned to 0 degrees
- moved D13 452.0 mm to (212.3, -66.9), turned to 0 degrees
- moved D23 448.9 mm to (212.3, -63.6), turned to 0 degrees
- moved D7 443.0 mm to (218.0, -70.3), turned to 0 degrees
- moved D25 437.7 mm to (212.3, -73.6), turned to 0 degrees
- moved R4 431.5 mm to (211.6, -60.4), turned to 0 degrees
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Connections:
- D10 pad 1: ROW2 -> ROW3
- D11 pad 1: ROW3 -> ROW0
- D12 pad 1: ROW0 -> ROW1
- D13 pad 1: Net-(D13-Pad1) -> ROW2
- D14 pad 1: ROW2 -> ROW3
- D15 pad 1: ROW3 -> ROW0
- D16 pad 1: ROW0 -> ROW1
- D17 pad 1: Net-(D13-Pad1) -> ROW2
- D18 pad 1: ROW2 -> ROW1
- D18 pad 2: Net-(D18-Pad2) -> COL4
- D19 pad 1: ROW3 -> ROW0
- D2 pad 1: Net-(D13-Pad1) -> ROW1
- D20 pad 1: Net-(D13-Pad1) -> ROW2
- D20 pad 2: COL4 -> Net-(D20-Pad2)
- D21 pad 1: ROW0 -> ROW3
- D22 pad 1: ROW2 -> ROW0
- D23 pad 1: ROW0 -> ROW1
- D24 pad 1: Net-(D24-Pad1) -> ROW2
- D25 pad 1: ROW2 -> ROW0
- D26 pad 1: ROW3 -> ROW1
- D27 pad 1: ROW0 -> ROW2
- D28 pad 1: Net-(D24-Pad1) -> ROW0
- D29 pad 1: ROW2 -> ROW1
- D30 pad 1: ROW0 -> ROW2
- D31 pad 1: Net-(D24-Pad1) -> ROW3
- D32 pad 1: ROW2 -> ROW0
- D33 pad 1: ROW0 -> ROW1
- D34 pad 1: Net-(D24-Pad1) -> ROW2
- D35 pad 1: ROW2 -> ROW0
- D36 pad 1: ROW0 -> ROW1
- D37 pad 1: Net-(D24-Pad1) -> ROW2
- D38 pad 1: ROW2 -> ROW3
- D39 pad 1: ROW3 -> ROW0
- D40 pad 1: ROW0 -> ROW1
- D41 pad 1: Net-(D24-Pad1) -> ROW2
- D42 pad 1: ROW2 -> ROW3
- D43 pad 1: ROW3 -> ROW0
- D45 pad 1: Net-(D24-Pad1) -> ROW2
- D46 pad 1: ROW2 -> ROW3
- D47 pad 1: ROW3 -> ROW0
- D48 pad 1: ROW0 -> ROW1
- D49 pad 1: Net-(D24-Pad1) -> ROW2
- D5 pad 1: Net-(D13-Pad1) -> ROW1
- D6 pad 1: ROW2 -> ROW3
- D7 pad 1: ROW3 -> ROW0
- D8 pad 1: ROW0 -> ROW1
- D9 pad 1: Net-(D13-Pad1) -> ROW2
- MX1 pad 3: Net-(MX1-Pad3) -> (no net)
- MX1 pad 4: Net-(MX1-Pad4) -> (no net)
- MX10 pad 3: Net-(MX10-Pad3) -> (no net)
- MX10 pad 4: Net-(MX10-Pad4) -> (no net)
- MX11 pad 1: COL2 -> COL3
- MX11 pad 3: Net-(MX11-Pad3) -> (no net)
- MX11 pad 4: Net-(MX11-Pad4) -> (no net)
- MX12 pad 3: Net-(MX12-Pad3) -> (no net)
- MX12 pad 4: Net-(MX12-Pad4) -> (no net)
- MX13 pad 3: Net-(MX13-Pad3) -> (no net)
- MX13 pad 4: Net-(MX13-Pad4) -> (no net)
- MX14 pad 3: Net-(MX14-Pad3) -> (no net)
- MX14 pad 4: Net-(MX14-Pad4) -> (no net)
- MX15 pad 1: COL3 -> COL4
- MX15 pad 3: Net-(MX15-Pad3) -> (no net)
- MX15 pad 4: Net-(MX15-Pad4) -> (no net)
- MX16 pad 3: Net-(MX16-Pad3) -> (no net)
- MX16 pad 4: Net-(MX16-Pad4) -> (no net)
- MX17 pad 1: COL4 -> ROW1
- MX17 pad 3: Net-(MX17-Pad3) -> (no net)
- MX17 pad 4: Net-(MX17-Pad4) -> (no net)
- MX18 pad 1: Net-(D13-Pad1) -> COL5
- MX18 pad 2: Net-(D18-Pad2) -> Net-(D19-Pad2)
- MX18 pad 3: Net-(MX18-Pad3) -> (no net)
- MX18 pad 4: Net-(MX18-Pad4) -> (no net)
- MX19 pad 1: Net-(D13-Pad1) -> COL5
- MX19 pad 2: Net-(D19-Pad2) -> Net-(MX19-Pad2)
- MX19 pad 3: Net-(MX19-Pad3) -> (no net)
- MX19 pad 4: Net-(MX19-Pad4) -> (no net)
- MX2 pad 3: Net-(MX2-Pad3) -> (no net)
- MX2 pad 4: Net-(MX2-Pad4) -> (no net)
- MX20 pad 2: Net-(D21-Pad2) -> Net-(D20-Pad2)
- MX20 pad 3: Net-(MX20-Pad3) -> (no net)
- MX20 pad 4: Net-(MX20-Pad4) -> (no net)
- MX21 pad 2: Net-(MX21-Pad2) -> Net-(D21-Pad2)
- MX21 pad 3: Net-(MX21-Pad3) -> (no net)
- MX21 pad 4: Net-(MX21-Pad4) -> (no net)
- MX22 pad 1: COL5 -> COL6
- MX22 pad 3: Net-(MX22-Pad3) -> (no net)
- MX22 pad 4: Net-(MX22-Pad4) -> (no net)
- MX23 pad 3: Net-(MX23-Pad3) -> (no net)
- MX23 pad 4: Net-(MX23-Pad4) -> (no net)
- MX24 pad 3: Net-(MX24-Pad3) -> (no net)
- MX24 pad 4: Net-(MX24-Pad4) -> (no net)
- MX25 pad 1: COL6 -> COL7
- MX25 pad 3: Net-(MX25-Pad3) -> (no net)
- MX25 pad 4: Net-(MX25-Pad4) -> (no net)
- MX26 pad 2: Net-(D27-Pad2) -> Net-(D26-Pad2)
- MX26 pad 3: Net-(MX26-Pad3) -> (no net)
- MX26 pad 4: Net-(MX26-Pad4) -> (no net)
- MX27 pad 2: Net-(D28-Pad2) -> Net-(D27-Pad2)
- MX27 pad 3: Net-(MX27-Pad3) -> (no net)
- MX27 pad 4: Net-(MX27-Pad4) -> (no net)
- MX28 pad 1: COL7 -> COL8
- MX28 pad 2: Net-(D29-Pad2) -> Net-(D28-Pad2)
- MX28 pad 3: Net-(MX28-Pad3) -> (no net)
- MX28 pad 4: Net-(MX28-Pad4) -> (no net)
- MX29 pad 1: COL7 -> COL8
- MX29 pad 2: Net-(D26-Pad2) -> Net-(D29-Pad2)
- MX29 pad 3: Net-(MX29-Pad3) -> (no net)
- MX29 pad 4: Net-(MX29-Pad4) -> (no net)
- MX3 pad 3: Net-(MX3-Pad3) -> (no net)
- MX3 pad 4: Net-(MX3-Pad4) -> (no net)
- MX30 pad 3: Net-(MX30-Pad3) -> (no net)
- MX30 pad 4: Net-(MX30-Pad4) -> (no net)
- MX31 pad 3: Net-(MX31-Pad3) -> (no net)
- MX31 pad 4: Net-(MX31-Pad4) -> (no net)
- MX32 pad 1: COL8 -> COL9
- MX32 pad 3: Net-(MX32-Pad3) -> (no net)
- MX32 pad 4: Net-(MX32-Pad4) -> (no net)
- MX33 pad 3: Net-(MX33-Pad3) -> (no net)
- MX33 pad 4: Net-(MX33-Pad4) -> (no net)
- MX34 pad 3: Net-(MX34-Pad3) -> (no net)
- MX34 pad 4: Net-(MX34-Pad4) -> (no net)
- MX35 pad 1: COL9 -> COL10
- MX35 pad 3: Net-(MX35-Pad3) -> (no net)
- MX35 pad 4: Net-(MX35-Pad4) -> (no net)
- MX36 pad 3: Net-(MX36-Pad3) -> (no net)
- MX36 pad 4: Net-(MX36-Pad4) -> (no net)
- MX37 pad 3: Net-(MX37-Pad3) -> (no net)
- MX37 pad 4: Net-(MX37-Pad4) -> (no net)
- MX38 pad 3: Net-(MX38-Pad3) -> (no net)
- MX38 pad 4: Net-(MX38-Pad4) -> (no net)
- MX39 pad 1: COL10 -> COL11
- MX39 pad 3: Net-(MX39-Pad3) -> (no net)
- MX39 pad 4: Net-(MX39-Pad4) -> (no net)
- MX4 pad 3: Net-(MX4-Pad3) -> (no net)
- MX4 pad 4: Net-(MX4-Pad4) -> (no net)
- MX40 pad 3: Net-(MX40-Pad3) -> (no net)
- MX40 pad 4: Net-(MX40-Pad4) -> (no net)
- MX41 pad 3: Net-(MX41-Pad3) -> (no net)
- MX41 pad 4: Net-(MX41-Pad4) -> (no net)
- MX42 pad 3: Net-(MX42-Pad3) -> (no net)
- MX42 pad 4: Net-(MX42-Pad4) -> (no net)
- MX43 pad 1: COL11 -> COL12
- MX43 pad 3: Net-(MX43-Pad3) -> (no net)
- MX43 pad 4: Net-(MX43-Pad4) -> (no net)
- MX45 pad 3: Net-(MX45-Pad3) -> (no net)
- MX45 pad 4: Net-(MX45-Pad4) -> (no net)
- MX46 pad 3: Net-(MX46-Pad3) -> (no net)
- MX46 pad 4: Net-(MX46-Pad4) -> (no net)
- MX47 pad 1: COL12 -> COL13
- MX47 pad 3: Net-(MX47-Pad3) -> (no net)
- MX47 pad 4: Net-(MX47-Pad4) -> (no net)
- MX48 pad 1: Net-(MX48-Pad1) -> COL13
- MX48 pad 3: Net-(MX48-Pad3) -> (no net)
- MX48 pad 4: Net-(MX48-Pad4) -> (no net)
- MX49 pad 1: Net-(MX49-Pad1) -> COL13
- MX49 pad 3: Net-(MX49-Pad3) -> (no net)
- MX49 pad 4: Net-(MX49-Pad4) -> (no net)
- MX5 pad 3: Net-(MX5-Pad3) -> (no net)
- MX5 pad 4: Net-(MX5-Pad4) -> (no net)
- MX50 pad 1: Net-(MX50-Pad1) -> COL14
- MX50 pad 3: Net-(MX50-Pad3) -> (no net)
- MX50 pad 4: Net-(MX50-Pad4) -> (no net)
- MX6 pad 3: Net-(MX6-Pad3) -> (no net)
- MX6 pad 4: Net-(MX6-Pad4) -> (no net)
- MX7 pad 1: COL1 -> COL2
- MX7 pad 3: Net-(MX7-Pad3) -> (no net)
- MX7 pad 4: Net-(MX7-Pad4) -> (no net)
- MX8 pad 3: Net-(MX8-Pad3) -> (no net)
- MX8 pad 4: Net-(MX8-Pad4) -> (no net)
- MX9 pad 3: Net-(MX9-Pad3) -> (no net)
- MX9 pad 4: Net-(MX9-Pad4) -> (no net)
- U1 pad 1: Net-(U1-Pad1) -> (no net)
- U1 pad 10: Net-(U1-Pad10) -> (no net)
- U1 pad 11: Net-(U1-Pad11) -> (no net)
- U1 pad 12: Net-(U1-Pad12) -> (no net)
- U1 pad 18: Net-(U1-Pad18) -> (no net)
- U1 pad 19: Net-(U1-Pad19) -> (no net)
- U1 pad 20: Net-(U1-Pad20) -> (no net)
- U1 pad 21: Net-(U1-Pad21) -> (no net)
- U1 pad 22: Net-(U1-Pad22) -> (no net)
- U1 pad 25: Net-(U1-Pad25) -> (no net)
- U1 pad 26: Net-(U1-Pad26) -> (no net)
- U1 pad 27: Net-(U1-Pad27) -> (no net)
- U1 pad 28: Net-(U1-Pad28) -> (no net)
- U1 pad 29: Net-(U1-Pad29) -> (no net)
- U1 pad 30: Net-(U1-Pad30) -> (no net)
- U1 pad 31: Net-(U1-Pad31) -> (no net)
- U1 pad 32: Net-(U1-Pad32) -> (no net)
- U1 pad 36: Net-(U1-Pad36) -> (no net)
- U1 pad 37: Net-(U1-Pad37) -> (no net)
- U1 pad 38: Net-(U1-Pad38) -> (no net)
- U1 pad 39: Net-(U1-Pad39) -> (no net)
- U1 pad 40: Net-(U1-Pad40) -> (no net)
- U1 pad 41: Net-(U1-Pad41) -> (no net)
- U1 pad 42: Net-(U1-Pad42) -> (no net)
- U1 pad 8: Net-(U1-Pad8) -> (no net)
- U1 pad 9: Net-(U1-Pad9) -> (no net)
- USB1 pad 2: Net-(USB1-Pad2) -> (no net)

Commit message: allign keyboard to grid
Parts:
- D1, D4: moved to B.Cu
- moved D4 199.9 mm to (49.2, 23.8), turned to 90 degrees
- moved D1 114.7 mm to (30.2, 23.8), turned to 90 degrees
- moved MX47 5.13 mm to (269.8, 23.8)
- moved MX48 5.06 mm to (262.7, 42.9)
- moved MX49 5.03 mm to (267.5, 61.9)
- moved MX43 4.76 mm to (250.8, 23.8)
- moved MX50 4.64 mm to (294.5, 23.8)
- moved MX40 4.63 mm to (236.5, 42.9)
- moved MX51 4.58 mm to (294.5, 42.9)
- moved MX39 4.40 mm to (231.7, 23.8)
- moved MX36 4.24 mm to (217.5, 42.9)
- moved MX35 4.05 mm to (212.7, 23.8)
- moved MX33 3.85 mm to (198.4, 42.9)
- moved MX32 3.70 mm to (193.6, 23.8)
- moved MX29 3.47 mm to (179.4, 42.9)
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
Commit message: align resistors with their keys
Parts:
- D10, D11, D12, D13, D14, D15, D16, D17, D18, D19, D2, D20, D21, D22, D23, D24, D25, D26, D27, D28, D29, D3, D30, D31, D32, D33, D34, D35, D36, D37, D38, D39, D40, D41, D42, D43, D45, D46, D47, D48, D49, D5, D50, D51, D6, D7, D8, D9: moved to B.Cu
- moved D50 275.4 mm to (302.4, 23.8), turned to 90 degrees
- moved D51 271.6 mm to (302.4, 42.9), turned to 90 degrees
- moved D49 265.4 mm to (275.4, 61.9), turned to 90 degrees
- moved D3 253.1 mm to (37.3, 61.9), turned to 90 degrees
- moved D2 244.2 mm to (32.5, 42.9), turned to 90 degrees
- moved D6 241.8 mm to (51.6, 81.0), turned to 90 degrees
- moved D48 234.5 mm to (270.7, 42.9), turned to 90 degrees
- moved D47 233.6 mm to (277.8, 23.8), turned to 90 degrees
- moved D46 219.2 mm to (256.4, 81.0), turned to 90 degrees
- moved D5 207.8 mm to (54.0, 42.9), turned to 90 degrees
- moved D45 205.6 mm to (254.0, 61.9), turned to 90 degrees
- moved D37 202.1 mm to (215.9, 61.9), turned to 90 degrees
- moved D43 197.4 mm to (258.8, 23.8), turned to 90 degrees
- moved D14 191.7 mm to (94.5, 81.0), turned to 90 degrees
- moved D17 191.0 mm to (101.6, 61.9), turned to 90 degrees
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
Commit message: clean up ratsnet
Parts:
- moved U1 196.3 mm to (289.7, 74.6)
- moved C5 194.9 mm to (299.6, 122.8)
- moved C6 194.9 mm to (268.9, 153.0)
- moved C1 194.9 mm to (225.2, 167.2)
- moved C2 194.9 mm to (229.6, 167.2)
- moved C3 194.9 mm to (234.0, 167.2)
- moved C4 194.9 mm to (238.4, 167.2)
- moved C7 194.9 mm to (299.6, 125.7)
- moved F1 194.9 mm to (319.4, 102.7)
- moved R1 194.9 mm to (293.8, 129.5)
- moved R2 194.9 mm to (349.3, 73.8)
- moved R3 194.9 mm to (340.8, 80.1)
- moved R4 194.9 mm to (323.5, 99.1)
- moved SW1 194.9 mm to (340.4, 65.4)
- moved USB1 194.9 mm to (343.5, 57.1)
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Connections:
- D14 pad 2: Net-(D14-Pad2) -> (no net)
- D18 pad 1: ROW1 -> ROW0
- D18 pad 2: COL4 -> Net-(D18-Pad2)
- D19 pad 1: ROW0 -> ROW1
- D21 pad 2: Net-(D21-Pad2) -> (no net)
- D40 pad 2: Net-(D40-Pad2) -> (no net)
- MX14 pad 1: COL3 -> COL4
- MX14 pad 2: Net-(D14-Pad2) -> Net-(MX14-Pad2)
- MX17 pad 1: ROW1 -> COL4
- MX18 pad 2: Net-(D19-Pad2) -> Net-(D18-Pad2)
- MX19 pad 2: Net-(MX19-Pad2) -> Net-(D19-Pad2)
- MX21 pad 2: Net-(D21-Pad2) -> Net-(MX21-Pad2)
- MX40 pad 2: Net-(D40-Pad2) -> Net-(MX40-Pad2)

Commit message: refine some alignment
Parts:
- U1: moved to B.Cu
- moved U1 9.15 mm to (292.5, 65.9)

Commit message: create PCB board outline
Parts:
- C1, C2, C3, C4, C5, C6, C7, R2, R3, R4, Y1: moved to B.Cu
- moved C1 102.3 mm to (294.0, 91.4), turned to 180 degrees
- moved C3 86.8 mm to (301.6, 112.6)
- moved C2 86.8 mm to (297.1, 112.6)
- moved C4 86.8 mm to (306.0, 112.6)
- moved C6 79.9 mm to (289.7, 75.9), turned to 270 degrees
- moved R2 63.5 mm to (287.6, 88.7), turned to 270 degrees
- moved R3 53.2 mm to (287.6, 81.0), turned to 90 degrees
- moved C5 46.9 mm to (298.4, 75.9), turned to 90 degrees
- moved C7 42.5 mm to (287.6, 84.9), turned to 270 degrees
- moved R4 24.9 mm to (302.4, 86.1), turned to 90 degrees
- moved R1 21.9 mm to (281.8, 111.1)
- moved D50 19.1 mm to (308.0, 42.1)
- moved D51 19.1 mm to (308.0, 61.1)
- moved MX50 19.1 mm to (300.0, 42.1)
- moved MX51 19.1 mm to (300.0, 61.1)
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Other:
- board outline added: 311.9 x 90.5 mm

Commit message: updated files
Parts:
- added D44: D, Diode_SMD:D_SOD-123, B.Cu at (56.0, 85.7)
- added D52: D, Diode_SMD:D_SOD-123, B.Cu at (289.3, 90.5)
- added D53: D, Diode_SMD:D_SOD-123, B.Cu at (308.4, 90.5)
- added D54: D, Diode_SMD:D_SOD-123, B.Cu at (310.8, 90.5)
- added MX41-1: MX-1.25U, MX_Alps_Hybrid:MXOnly-1.25U-NoLED, F.Cu at (254.8, 66.7)
- added MX42-1: MX-1U, MX_Alps_Hybrid:MXOnly-1U-NoLED, F.Cu at (276.2, 66.7)
- added MX44: MX-1U, MX_Alps_Hybrid:MXOnly-1U-NoLED, F.Cu at (47.6, 85.7)
- added MX52: MX-1U, MX_Alps_Hybrid:MXOnly-1U-NoLED, F.Cu at (281.0, 90.5)
- added MX53: MX-1U, MX_Alps_Hybrid:MXOnly-1U-NoLED, F.Cu at (300.0, 90.5)
- added MX54: MX-1U, MX_Alps_Hybrid:MXOnly-1U-NoLED, F.Cu at (319.1, 90.5)
- D1, D10, D11, D12, D13, D14, D15, D16, D17, D18, D19, D2, D20, D21, D22, D23, D24, D25, D26, D27, D28, D29, D3, D30, D31, D32, D33, D34, D35, D36, D37, D38, D39, D4, D40, D41, D42, D43, D45, D46, D47, D48, D49, D5, D50, D51, D6, D7, D8, D9: value SOD-123 -> D
- F1, SW1: moved to B.Cu
- MX1, MX10, MX11, MX12, MX13, MX15, MX17, MX18, MX19, MX20, MX22, MX23, MX24, MX25, MX26, MX27, MX29, MX32, MX33, MX34, MX35, MX36, MX37, MX39, MX4, MX40, MX41, MX43, MX5, MX51, MX7, MX8, MX9: footprint MX_Alps_Hybrid:MX-1U -> MX_Alps_Hybrid:MXOnly-1U-NoLED
- MX14, MX2, MX38, MX6: value MX-1.25U -> MX-1U; footprint MX_Alps_Hybrid:MX-1.25U -> MX_Alps_Hybrid:MXOnly-1U-NoLED
- MX16, MX42, MX45, MX50: value MX-1U -> MX-1.25U; footprint MX_Alps_Hybrid:MX-1U -> MX_Alps_Hybrid:MXOnly-1.25U-NoLED
- MX21: value MX-2.25U -> MX-1U; footprint MX_Alps_Hybrid:MX-2.25U -> MX_Alps_Hybrid:MXOnly-1U-NoLED
- MX28, MX30: value MX-1U -> MX-1.75U; footprint MX_Alps_Hybrid:MX-1U -> MX_Alps_Hybrid:MXOnly-1.75U-NoLED
- MX3: value MX-1.75U -> MX-1U; footprint MX_Alps_Hybrid:MX-1.75U -> MX_Alps_Hybrid:MXOnly-1U-NoLED
- MX31: value MX-2.75U -> MX-1U; footprint MX_Alps_Hybrid:MX-2.75U -> MX_Alps_Hybrid:MXOnly-1U-NoLED
- MX46, MX49: footprint MX_Alps_Hybrid:MX-1.25U -> MX_Alps_Hybrid:MXOnly-1.25U-NoLED
- MX47: value MX-1U -> MX-2.25U; footprint MX_Alps_Hybrid:MX-1U -> MX_Alps_Hybrid:MXOnly-2.25U-ReversedStabilizers-NoLED
- MX48: value MX-1.75U -> MX-2.75U; footprint MX_Alps_Hybrid:MX-1.75U -> MX_Alps_Hybrid:MXOnly-2.75U-ReversedStabilizers-NoLED
- R1: value 22 -> 10k; moved to B.Cu
- R3: value 10k -> 22
- U1: value ATmega32U4-MU -> ATmega32U4-AU; footprint Package_QFP:TQFP-48-1EP_7x7mm_P0.5mm_EP3.5x3.5mm -> Package_QFP:TQFP-44_10x10mm_P0.8mm
- USB1: value Molex-0548190589 -> USB Mini; footprint random-keyboard-parts:Molex-0548190589 -> local:USB-Mini-B_ LCSC-C46398
- moved D14 200.6 mm to (284.6, 28.6)
- moved MX14 200.2 mm to (276.2, 28.6)
- moved USB1 200.0 mm to (152.4, 25.0), turned to 180 degrees
- moved MX15 199.7 mm to (300.0, 28.6)
- moved F1 192.5 mm to (150.2, 33.6), turned to 90 degrees
- moved D13 187.8 mm to (265.5, 28.6)
- moved MX13 187.5 mm to (257.2, 28.6)
- moved D15 183.5 mm to (291.7, 28.6)
- moved MX45 179.4 mm to (69.1, 85.7)
- moved D45 179.1 mm to (77.4, 85.7)
- moved MX46 158.5 mm to (92.9, 85.7)
- moved D46 158.1 mm to (101.2, 85.7)
- moved D12 155.4 mm to (246.5, 28.6)
- moved MX12 155.1 mm to (238.1, 28.6)
- moved MX47 152.4 mm to (126.2, 85.7)
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Connections:
- net Net-(C5-Pad1) renamed /XT1
- net Net-(C6-Pad1) renamed /XT2
- net Net-(R2-Pad1) renamed /MCU_D+
- D1 pad 1: ROW0 -> row0
- D10 pad 1: ROW3 -> row0
- D11 pad 1: ROW0 -> row0
- D12 pad 1: ROW1 -> row0
- D13 pad 1: ROW2 -> row0
- D14 pad 1: ROW3 -> row0
- D14 pad 2: (no net) -> Net-(D14-Pad2)
- D15 pad 1: ROW0 -> row0
- D16 pad 1: ROW1 -> row1
- D17 pad 1: ROW2 -> row1
- D18 pad 1: ROW0 -> row1
- D19 pad 1: ROW1 -> row1
- D2 pad 1: ROW1 -> row0
- D20 pad 1: ROW2 -> row1
- D21 pad 1: ROW3 -> row1
- D21 pad 2: (no net) -> Net-(D21-Pad2)
- D22 pad 1: ROW0 -> row1
- D23 pad 1: ROW1 -> row1
- D24 pad 1: ROW2 -> row1
- D25 pad 1: ROW0 -> row1
- D26 pad 1: ROW1 -> row1
- D27 pad 1: ROW2 -> row1
- D28 pad 1: ROW0 -> row1
- D29 pad 1: ROW1 -> row1
- D3 pad 1: ROW2 -> row0
- D30 pad 1: ROW2 -> row2
- D31 pad 1: ROW3 -> row2
- D32 pad 1: ROW0 -> row2
- D33 pad 1: ROW1 -> row2
- D34 pad 1: ROW2 -> row2
- D35 pad 1: ROW0 -> row2
- D36 pad 1: ROW1 -> row2
- D37 pad 1: ROW2 -> row2
- D38 pad 1: ROW3 -> row2
- D39 pad 1: ROW0 -> row2
- D4 pad 1: ROW0 -> row0
- D40 pad 1: ROW1 -> row2
- D40 pad 2: (no net) -> Net-(D40-Pad2)
- D41 pad 1: ROW2 -> row2
- D42 pad 1: ROW3 -> row2
- D43 pad 1: ROW0 -> row2
- D45 pad 1: ROW2 -> row3
- D46 pad 1: ROW3 -> row3
- D47 pad 1: ROW0 -> row3
- D48 pad 1: ROW1 -> row3
- D49 pad 1: ROW2 -> row3
- D5 pad 1: ROW1 -> row0
- D50 pad 1: ROW0 -> row3
- D51 pad 1: ROW1 -> row3
- D6 pad 1: ROW3 -> row0
- D7 pad 1: ROW0 -> row0
- D8 pad 1: ROW1 -> row0
- D9 pad 1: ROW2 -> row0
- MX1 pad 1: COL0 -> colA
- MX10 pad 1: COL2 -> colJ
- MX11 pad 1: COL3 -> colK
- MX12 pad 1: COL3 -> colL
- MX13 pad 1: COL3 -> colM
- MX14 pad 1: COL4 -> colN
- MX14 pad 2: Net-(MX14-Pad2) -> Net-(D14-Pad2)
- MX15 pad 1: COL4 -> Net-(D15-Pad2)
- MX15 pad 2: Net-(D15-Pad2) -> colO
- MX16 pad 1: COL4 -> colA
- MX17 pad 1: COL4 -> colB
- MX18 pad 1: COL5 -> colC
- MX19 pad 1: COL5 -> colD
- MX2 pad 1: COL0 -> colB
- MX20 pad 1: COL5 -> colE
- MX21 pad 1: COL5 -> colF
- MX21 pad 2: Net-(MX21-Pad2) -> Net-(D21-Pad2)
- MX22 pad 1: COL6 -> colG
- MX23 pad 1: COL6 -> colH
- MX24 pad 1: COL6 -> colI
- MX25 pad 1: COL7 -> colJ
- MX26 pad 1: COL7 -> colK
- MX27 pad 1: COL7 -> colL
- MX28 pad 1: COL8 -> colM
- MX29 pad 1: COL8 -> Net-(D29-Pad2)
- MX29 pad 2: Net-(D29-Pad2) -> colO
- MX3 pad 1: COL0 -> colC
- MX30 pad 1: COL8 -> colA
- MX31 pad 1: COL8 -> colB
- MX32 pad 1: COL9 -> colC
- MX33 pad 1: COL9 -> colD
- MX34 pad 1: COL9 -> colE
- MX35 pad 1: COL10 -> colF
- MX36 pad 1: COL10 -> colG
- MX37 pad 1: COL10 -> colH
- MX38 pad 1: COL10 -> colI
- MX39 pad 1: COL11 -> colJ
- MX4 pad 1: COL1 -> colD
- MX40 pad 1: COL11 -> colK
- MX40 pad 2: Net-(MX40-Pad2) -> Net-(D40-Pad2)
- MX41 pad 1: COL11 -> colL
- MX42 pad 1: COL11 -> Net-(D42-Pad2)
- MX42 pad 2: Net-(D42-Pad2) -> colN
- MX43 pad 1: COL12 -> Net-(D43-Pad2)
- MX43 pad 2: Net-(D43-Pad2) -> colO
- MX45 pad 1: COL12 -> colB
- MX46 pad 1: COL12 -> colD
- MX47 pad 1: COL13 -> colE
- MX48 pad 1: COL13 -> colH
- MX49 pad 1: COL13 -> colJ
- MX5 pad 1: COL1 -> colE
- MX50 pad 1: COL14 -> colK
- MX51 pad 1: COL14 -> colL
- MX6 pad 1: COL1 -> colF
- MX7 pad 1: COL2 -> colG
- MX8 pad 1: COL2 -> colH
- MX9 pad 1: COL2 -> colI
- R1 pad 1: Net-(R1-Pad1) -> +5V
- R1 pad 2: D- -> Net-(R1-Pad2)
- R3 pad 1: +5V -> /MCU_D-
- R3 pad 2: Net-(R3-Pad2) -> D-
- SW1 pad 2: Net-(R3-Pad2) -> Net-(R1-Pad2)
- U1 pad 1: (no net) -> Net-(U1-Pad1)
- U1 pad 10: (no net) -> Net-(U1-Pad10)
- U1 pad 11: (no net) -> Net-(U1-Pad11)
- U1 pad 12: (no net) -> Net-(U1-Pad12)
- U1 pad 13: Net-(R3-Pad2) -> Net-(R1-Pad2)
- U1 pad 18: (no net) -> colO
- U1 pad 19: (no net) -> row3
- U1 pad 20: (no net) -> colN
- U1 pad 21: (no net) -> colM
- U1 pad 22: (no net) -> colL
- U1 pad 25: (no net) -> colK
- U1 pad 26: (no net) -> colJ
- U1 pad 27: (no net) -> colH
- U1 pad 28: (no net) -> colE
- U1 pad 29: (no net) -> colD
- U1 pad 3: Net-(R1-Pad1) -> /MCU_D-
- U1 pad 30: (no net) -> colB
- U1 pad 31: (no net) -> colA
- U1 pad 32: (no net) -> row2
- U1 pad 36: (no net) -> Net-(U1-Pad36)
- U1 pad 37: (no net) -> colI
- U1 pad 38: (no net) -> colG
- U1 pad 39: (no net) -> colF
- U1 pad 40: (no net) -> colC
- U1 pad 41: (no net) -> row1
- U1 pad 42: (no net) -> Net-(U1-Pad42)
- U1 pad 8: (no net) -> row0
- U1 pad 9: (no net) -> Net-(U1-Pad9)
- USB1 pad 2: (no net) -> Net-(USB1-Pad2)
- USB1 pad 6: Net-(USB1-Pad6) -> GND
Routing:
- net colA: track 0.00 -> 356.2 mm, vias 0 -> 1
- net colB: track 0.00 -> 331.4 mm, vias 0 -> 1
- net row0: track 0.00 -> 300.5 mm, vias 0 -> 2
- net row3: track 0.00 -> 300.1 mm
- net colD: track 0.00 -> 293.7 mm, vias 0 -> 1
- net GND: track 0.00 -> 288.5 mm
- net row2: track 0.00 -> 285.4 mm
- net colC: track 0.00 -> 281.7 mm, vias 0 -> 1
- net row1: track 0.00 -> 273.9 mm
- net colE: track 0.00 -> 273.8 mm, vias 0 -> 1
- net +5V: track 0.00 -> 239.4 mm, vias 0 -> 4
- net colF: track 0.00 -> 224.8 mm, vias 0 -> 1
- net colH: track 0.00 -> 217.0 mm, vias 0 -> 1
- net colG: track 0.00 -> 205.6 mm, vias 0 -> 1
- net colJ: track 0.00 -> 177.9 mm, vias 0 -> 1
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- added copper zone on B.Cu, net GND
Other:
- board size 311.9 x 90.5 mm -> 307.2 x 79.8 mm
- net class Default: clearance 0.2 -> 0.17; via_dia 0.8 -> 0.6; via_drill 0.4 -> 0.3
- net class Primary added: clearance 0.19, trace_width 0.381, via_dia 0.8, via_drill 0.4
- net class Signal added: clearance 0.16256, trace_width 0.2032, via_dia 0.6, via_drill 0.3
- rule trace_clearance: 0.2 -> 0.17
