File: pcb/CoquiReplacement.kicad_pcb (KiCad board)
At the start: 2 copper layers, 307.2 x 79.8 mm, 128 parts, among them P1 USB_C_Plug_USB2.0, SW1 SW_Push, U1 ATmega32U4-AU, Y1 16MHz

Commit message: cleanup
Parts:
- MX9: moved to F.Cu
- turned MX9 to 0 degrees
Changed lines of the file:
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@@
     (pad "" np_thru_hole circle (at 5.08 0 48.0996) (size 1.75 1.75) (drill 1.75) (layers *.Cu *.Mask))
   )
-  (module MX_Alps_Hybrid:MXOnly-1U-NoLED (layer B.Cu)
-    (at 66.675 28.575 180)
-    (fp_text reference MX9 (at 0 -3.175) (layer Dwgs.User)
-      (effects (font (size 1 1) (thickness 0.15)))
-    )
-    (fp_text value MX-1U (at 0 7.9375) (layer Dwgs.User)
-      (effects (font (size 1 1) (thickness 0.15)))
-    )
-    (fp_line (start 5 7) (end 7 7) (layer Dwgs.User) (width 0.15))
-    (fp_line (start 7 7) (end 7 5) (layer Dwgs.User) (width 0.15))
-    (fp_line (start 5 -7) (end 7 -7) (layer Dwgs.User) (width 0.15))
-    (fp_line (start 7 -7) (end 7 -5) (layer Dwgs.User) (width 0.15))
-    (fp_line (start -7 -5) (end -7 -7) (layer Dwgs.User) (width 0.15))
-    (fp_line (start -7 -7) (end -5 -7) (layer Dwgs.User) (width 0.15))
-    (fp_line (start -5 7) (end -7 7) (layer Dwgs.User) (width 0.15))
-    (fp_line (start -7 7) (end -7 5) (layer Dwgs.User) (width 0.15))
-    (fp_line (start -9.525 9.525) (end 9.525 9.525) (layer Dwgs.User) (width 0.15))
-    (fp_line (start 9.525 9.525) (end 9.525 -9.525) (layer Dwgs.User) (width 0.15))
-    (fp_line (start 9.525 -9.525) (end -9.525 -9.525) (layer Dwgs.User) (width 0.15))
-    (fp_line (start -9.525 -9.525) (end -9.525 9.525) (layer Dwgs.User) (width 0.15))
-    (pad 2 thru_hole circle (at 2.54 5.08 180) (size 2.25 2.25) (drill 1.47) (layers *.Cu F.Mask)
+  (module MX_Alps_Hybrid:MXOnly-1U-NoLED (layer F.Cu)
+    (at 66.675 28.575)
+    (fp_text reference MX9 (at 0 3.175 -90) (layer Dwgs.User)
+      (effects (font (size 1 1) (thickness 0.15)))
+    )
+    (fp_text value MX-1U (at 0 -7.9375 180) (layer Dwgs.User)
+      (effects (font (size 1 1) (thickness 0.15)))
+    )
+    (fp_line (start 5 -7) (end 7 -7) (layer Dwgs.User) (width 0.15))
+    (fp_line (start 7 -7) (end 7 -5) (layer Dwgs.User) (width 0.15))
+    (fp_line (start 5 7) (end 7 7) (layer Dwgs.User) (width 0.15))
+    (fp_line (start 7 7) (end 7 5) (layer Dwgs.User) (width 0.15))
+    (fp_line (start -7 5) (end -7 7) (layer Dwgs.User) (width 0.15))
+    (fp_line (start -7 7) (end -5 7) (layer Dwgs.User) (width 0.15))
+    (fp_line (start -5 -7) (end -7 -7) (layer Dwgs.User) (width 0.15))
+    (fp_line (start -7 -7) (end -7 -5) (layer Dwgs.User) (width 0.15))
+    (fp_line (start -9.525 -9.525) (end 9.525 -9.525) (layer Dwgs.User) (width 0.15))
+    (fp_line (start 9.525 -9.525) (end 9.525 9.525) (layer Dwgs.User) (width 0.15))
+    (fp_line (start 9.525 9.525) (end -9.525 9.525) (layer Dwgs.User) (width 0.15))
+    (fp_line (start -9.525 9.525) (end -9.525 -9.525) (layer Dwgs.User) (width 0.15))
+    (pad 2 thru_hole circle (at 2.54 -5.08) (size 2.25 2.25) (drill 1.47) (layers *.Cu B.Mask)
       (net 12 "Net-(D9-Pad2)"))
-    (pad "" np_thru_hole circle (at 0 0 180) (size 3.9878 3.9878) (drill 3.9878) (layers *.Cu *.Mask))
-    (pad 1 thru_hole circle (at -3.81 2.54 180) (size 2.25 2.25) (drill 1.47) (layers *.Cu F.Mask)
+    (pad "" np_thru_hole circle (at 0 0) (size 3.9878 3.9878) (drill 3.9878) (layers *.Cu *.Mask))
+    (pad 1 thru_hole circle (at -3.81 -2.54) (size 2.25 2.25) (drill 1.47) (layers *.Cu B.Mask)
       (net 71 colC))
-    (pad "" np_thru_hole circle (at -5.08 0 131.9004) (size 1.75 1.75) (drill 1.75) (layers *.Cu *.Mask))
-    (pad "" np_thru_hole circle (at 5.08 0 131.9004) (size 1.75 1.75) (drill 1.75) (layers *.Cu *.Mask))
+    (pad "" np_thru_hole circle (at -5.08 0 48.0996) (size 1.75 1.75) (drill 1.75) (layers *.Cu *.Mask))
+    (pad "" np_thru_hole circle (at 5.08 0 48.0996) (size 1.75 1.75) (drill 1.75) (layers *.Cu *.Mask))
   )
   (module MX_Alps_Hybrid:MXOnly-1U-NoLED (layer F.Cu)
@@
   (segment (start 50.1396 23.5204) (end 50.165 23.495) (width 0.25) (layer B.Cu) (net 8))
   (segment (start 50.1396 34.8508) (end 50.1396 23.5204) (width 0.25) (layer B.Cu) (net 8))
-  (segment (start 55.959375 26.2718) (end 55.959375 26.925) (width 0.2032) (layer B.Cu) (net 85))
   (segment (start 60.721875 45.3218) (end 60.721875 45.975) (width 0.2032) (layer B.Cu) (net 9))
   (segment (start 57.945075 42.545) (end 60.721875 45.3218) (width 0.2032) (layer B.Cu) (net 9))
@@
   (segment (start 318.16908 59.903592) (end 318.16908 63.386256) (width 0.2032) (layer B.Cu) (net 83))
   (via (at 310.157948 83.939008) (size 0.6) (drill 0.3) (layers F.Cu B.Cu) (net 83))
+  (segment (start 55.959375 26.2718) (end 55.959375 26.925) (width 0.2032) (layer B.Cu) (net 85))
   (segment (start 315.559912 54.247624) (end 317.227096 54.247624) (width 0.25) (layer B.Cu) (net 86))
   (segment (start 317.227096 54.247624) (end 317.598968 53.875752) (width 0.25) (layer B.Cu) (net 86))
